File: doc/example_board/IoT_Led_v1.kicad_sch (KiCad schematic)
At the start: 66 parts, among them J1 LEDs, J2 USB, J3 Barrel_Jack_PTH_Slot, Q1 AON7466, Q10 IRF540N, Q11 AOI4184, Q12 2N7000/2N5550, Q13 AON7466, Q14 IRF540N, Q15 AOI4184, Q16 2N7000/2N5550, Q2 IRF540N, Q3 AOI4184, Q4 2N7000/2N5550, Q5 AON7466, Q6 IRF540N, Q7 AOI4184, Q8 2N7000/2N5550, Q9 AON7466, U1 LD1117V33, U2 MC34063AP, U3 ESP32-C3-WROOM-02

Commit message: Upgrading the example board
Changed lines of the file:
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@@
 		)
 	)
-	(text "Output modes:\nAll power transistors should be the same.\nChoose (Q1, Q5, Q9, Q13), (Q2, Q6, Q10, Q14) or (Q3, Q7, Q11, Q15)\nIf the power transistor is saturated for the projected current \nwhen V_gs = 3.3V use the inversion. To use the inversion:\n* open JP1, JP5, JP6, JP8;\n* insert R1, Q4, R6, Q8, R11, Q12, R13, Q16.\nFor non-inverting mode, close the jumpers \nand do not insert elements listed above.\nFor three-channel output, just skip any output section.\n\nPower modes:\nPossible configurations:\n* Pulse regulator and no linear regulator - close JP2, skip U1.\n* Pulse regulator and linear regulator - close JP3, skip R5 and R6.\n* No pulse regulator and linear regulator - close JP4, skip \n  all parts of \"Pulse regulator\".\n\nResistors:\nAll resistors without given values should be the same \nand have a value between 1kOhm and 4.7kOhm"
+	(text "Output modes:\nAll power transistors should be the same.\nChoose (Q1, Q5, Q9, Q13), (Q2, Q6, Q10, Q14) or (Q3, Q7, Q11, Q15)\nIf the power transistor is saturated for the projected current \nwhen V_gs = 3.3V use the inversion. To use the inversion:\n* open JP1, JP5, JP6, JP8;\n* insert R1, Q4, R6, Q8, R11, Q12, R13, Q16.\nFor non-inverting mode, close the jumpers \nand do not insert elements listed above.\nFor three-channel output, just skip any output section.\n\nUse D2, D4, D7 and D9 only when using invert mode and\nV_gs breakout is not greater than V_in (12V) * 125%.\n\nPower modes:\nPossible configurations:\n* Pulse regulator and no linear regulator - close JP2, skip U1.\n* Pulse regulator and linear regulator - close JP3, skip R5 and R8 \n  or skip only R7. The option with skipping R7 is recommended.\n* No pulse regulator and linear regulator - close JP4, skip \n  all parts of \"Pulse regulator\".\n\nResistors:\nAll resistors without given values should be the same \nand have a value between 1kOhm and 4.7kOhm\n"
 		(exclude_from_sim no)
-		(at 111.506 168.402 0)
+		(at 111.76 172.466 0)
 		(effects
 			(font
@@
 	)
 	(junction
-		(at 67.31 19.05)
-		(diameter 0)
-		(color 0 0 0 0)
-	)
-	(junction
 		(at 77.47 191.77)
 		(diameter 0)
@@
 	)
 	(junction
-		(at 67.31 111.76)
-		(diameter 0)
-		(color 0 0 0 0)
-	)
-	(junction
 		(at 48.26 66.04)
 		(diameter 0)
@@
 	)
 	(junction
-		(at 67.31 66.04)
-		(diameter 0)
-		(color 0 0 0 0)
-	)
-	(junction
 		(at 58.42 100.33)
 		(diameter 0)
@@
 	)
 	(junction
-		(at 67.31 157.48)
-		(diameter 0)
-		(color 0 0 0 0)
-	)
-	(junction
 		(at 48.26 111.76)
 		(diameter 0)
@@
 	(wire
 		(pts
-			(xy 67.31 19.05) (xy 58.42 19.05)
+			(xy 58.42 19.05) (xy 67.31 19.05)
 		)
 		(stroke
@@
 	(wire
 		(pts
-			(xy 68.58 66.04) (xy 67.31 66.04)
-		)
-		(stroke
-			(width 0)
-			(type default)
-		)
-	)
-	(wire
-		(pts
 			(xy 95.25 76.2) (xy 97.79 76.2)
 		)
@@
 	(wire
 		(pts
-			(xy 68.58 157.48) (xy 67.31 157.48)
-		)
-		(stroke
-			(width 0)
-			(type default)
-		)
-	)
-	(wire
-		(pts
 			(xy 77.47 34.29) (xy 77.47 41.91)
 		)
@@
 	(wire
 		(pts
-			(xy 67.31 66.04) (xy 58.42 66.04)
+			(xy 58.42 66.04) (xy 67.31 66.04)
 		)
 		(stroke
@@
 	(wire
 		(pts
-			(xy 67.31 111.76) (xy 58.42 111.76)
+			(xy 58.42 111.76) (xy 67.31 111.76)
 		)
 		(stroke
@@
 	(wire
 		(pts
-			(xy 68.58 111.76) (xy 67.31 111.76)
-		)
-		(stroke
-			(width 0)
-			(type default)
-		)
-	)
-	(wire
-		(pts
 			(xy 85.09 93.98) (xy 97.79 93.98)
 		)
@@
 	(wire
 		(pts
-			(xy 196.85 142.24) (xy 210.82 142.24)
+			(xy 200.66 142.24) (xy 210.82 142.24)
 		)
 		(stroke
@@
 	(wire
 		(pts
-			(xy 68.58 19.05) (xy 67.31 19.05)
-		)
-		(stroke
-			(width 0)
-			(type default)
-		)
-	)
-	(wire
-		(pts
 			(xy 48.26 177.8) (xy 48.26 191.77)
 		)
@@
 	(wire
 		(pts
-			(xy 67.31 157.48) (xy 58.42 157.48)
+			(xy 58.42 157.48) (xy 67.31 157.48)
 		)
 		(stroke
@@
 	(global_label "12V"
 		(shape output)
-		(at 196.85 142.24 180)
+		(at 200.66 142.24 180)
 		(fields_autoplaced yes)
 		(effects
@@
 		)
 		(property "Intersheetrefs" "${INTERSHEET_REFS}"
-			(at 190.3572 142.24 0)
+			(at 194.1672 142.24 0)
 			(effects
 				(font
@@
 		(dnp no)
 		(property "Reference" "J3"
-			(at 265.938 138.176 0)
+			(at 263.398 138.43 0)
 			(effects
 				(font
@@
 		)
 		(property "Value" "Barrel_Jack_PTH_Slot"
-			(at 265.938 141.224 0)
+			(at 263.398 140.97 0)
 			(effects
 				(font

Commit message: Board upgrade
Parts:
- added J4: FAN, Connector_PinSocket_2.54mm:PinSocket_2x02_P2.54mm_Vertical, symbol PCM_SL_Pin_Headers:PINHD_2x2_Female
- added Q17: 2N7000/2N5550, Package_TO_SOT_THT:TO-92_Inline, symbol Transistor_FET:2N7000
Connections:
- net 12V: now also J4.3
- net GND: now also Q17.1 (S)
- net at U3.10 (IO10), U3.12 (IO21/TXD): now also Q17.2 (G)
- net Vmid: now reaches C4.1, JP2.2 (B), JP3.2 (B), L1.1, R5.2, R7.2
- net Vmid: now also J4.1
- new net: J4.2, J4.4, Q17.3 (D)
Other:
- moved on the sheet: C10, C6, C7, C8, C9, J3

Commit message: Board update
Parts:
- added C11: 1u, Capacitor_THT:C_Disc_D3.0mm_W2.0mm_P2.50mm, symbol PCM_SL_Devices:Capacitor_NP
- added Q18: 2N5550, Package_TO_SOT_THT:TO-92_Inline, symbol Transistor_BJT:2N3904
- C5: value 470p -> 47p-470p
- D6: value 1N4002 -> 1n5819
- L1: value 100u-500u -> 47u-470u
Connections:
- net GND: now also C11.1, Q18.2 (B), Q18.3 (C)
- net Vmid: now also C11.2
- net at D6.1 (K), L1.2, U2.2 (SwE): now also Q18.1 (E)
Other:
- note added: "D6 or Q18, not both D6 is strongly recommended"
- note added: "L1/[uH] ~= C5/[pF]"
- moved on the sheet: C4

Commit message: Board update - added a capacitor and a resistor for CHP_EN, added a rst pad
Parts:
- added C12: 1u, Capacitor_THT:C_Disc_D3.0mm_W2.0mm_P2.50mm, symbol PCM_SL_Devices:Capacitor_NP
- added JP9: RST, PCM_SparkFun-Jumper:Jumper_2_NO_NoSilk, symbol PCM_SparkFun-Jumper:SolderJumper_2_Open_No_Silk
- added R14: R, Resistor_THT:R_Axial_DIN0207_L6.3mm_D2.5mm_P10.16mm_Horizontal, symbol PCM_SL_Resistors:Resistor
- D1, D3, D5, D8: value 1N4002 -> 1n5819
Connections:
- net 3V3: now also R14.1; no longer U3.2 (EN)
- net GND: now also C12.1, JP9.2 (B)
- new net: C12.2, JP9.1 (A), R14.2, U3.2 (EN)
