File: doc/example_board/IoT_Led_v1.kicad_pcb (KiCad board)
At the start: 2 copper layers, 80 x 60 mm, 66 parts, among them J1 LEDs, J2 USB, J3 Barrel_Jack_PTH_Slot, Q1 AON7466, Q10 IRF540N, Q11 AOI4184, Q12 2N7000/2N5550, Q13 AON7466, Q14 IRF540N, Q15 AOI4184, Q16 2N7000/2N5550, Q2 IRF540N, Q3 AOI4184, Q4 2N7000/2N5550, Q5 AON7466, Q6 IRF540N, Q7 AOI4184, Q8 2N7000/2N5550, Q9 AON7466, U1 LD1117V33, U2 MC34063AP, U3 ESP32-C3-WROOM-02

Commit message: Upgrading the example board
Parts:
- moved JP4 1.61 mm to (133.6, 84.0)
- moved R10 1.19 mm to (119.6, 91.5)
- moved R2 0.08 mm to (118.0, 121.1)
Routing:
- net 12V: track 159.4 -> 191.4 mm
- net Net-(C1-Pad2): track 59.4 -> 74.9 mm
- net Net-(JP5-A): track 41.4 -> 46.8 mm, vias 0 -> 1
- net Net-(JP6-A): track 53.8 -> 57.1 mm, vias 0 -> 1
- net Net-(JP8-A): track 65.0 -> 67.2 mm, vias 0 -> 1
- net Net-(JP1-A): track 40.2 -> 38.5 mm
- net Net-(U3-IO3): track 95.1 -> 96.7 mm
- net Net-(JP3-A): track 12.4 -> 10.9 mm
- net Net-(U3-IO2): track 112.1 -> 110.8 mm
- net Net-(U2-Vfb): track 24.9 -> 24.0 mm
- net Net-(U3-IO4): track 62.0 -> 61.4 mm
- net 3V3: track 73.5 -> 74.1 mm
- net GND: vias 36 -> 134

Commit message: Board upgrade
Parts:
- added J4: FAN, Connector_PinSocket_2.54mm:PinSocket_2x02_P2.54mm_Vertical, F.Cu at (128.3, 93.2)
- added Q17: 2N7000/2N5550, Package_TO_SOT_THT:TO-92_Inline, F.Cu at (118.5, 94.6)
- moved C1 5.26 mm to (118.0, 102.0), turned to 90 degrees
- moved R10 2.06 mm to (120.7, 89.8)
Connections:
- net Net-(JP2-B) renamed Vmid
Routing:
- net Net-(Q17-G): track 6.27 -> 65.5 mm, vias 0 -> 1
- net GND: track 37.5 -> 60.4 mm, vias 134 -> 124
- net Vmid: track 53.8 -> 72.1 mm, vias 0 -> 1
- net Net-(Q17-D): track 0.00 -> 10.5 mm
- net 12V: track 191.4 -> 199.8 mm
- net 3V3: track 74.1 -> 76.0 mm
- net Net-(U2-Vfb): track 24.0 -> 22.5 mm
- net Net-(JP5-A): track 46.8 -> 46.0 mm

Commit message: Board update
Parts:
- added C11: 1u, Capacitor_THT:C_Disc_D3.0mm_W2.0mm_P2.50mm, F.Cu at (119.8, 77.8)
- added Q18: 2N5550, Package_TO_SOT_THT:TO-92_Inline, F.Cu at (118.1, 81.7)
- C5: value 470p -> 47p-470p
- D6: value 1N4002 -> 1n5819
- L1: value 100u-500u -> 47u-470u
- moved C5 2.44 mm to (117.2, 87.0), turned to 0 degrees
- moved D6 1.13 mm to (113.8, 83.2)
Routing:
- net Net-(D6-K): track 12.4 -> 16.4 mm
- net Vmid: track 72.1 -> 74.8 mm
- net GND: track 60.4 -> 61.6 mm, vias 124 -> 142
- net Net-(U2-TC): track 3.07 -> 4.13 mm

Commit message: Board update - added a capacitor and a resistor for CHP_EN, added a rst pad
Parts:
- added C12: 1u, Capacitor_THT:C_Disc_D3.0mm_W2.0mm_P2.50mm, F.Cu at (144.0, 73.5)
- added JP9: RST, PCM_SparkFun-Jumper:Jumper_2_NO_NoSilk, F.Cu at (138.5, 83.0)
- added R14: R, Resistor_THT:R_Axial_DIN0207_L6.3mm_D2.5mm_P10.16mm_Horizontal, F.Cu at (132.8, 76.5)
- D1, D3, D5, D8: value 1N4002 -> 1n5819
- moved R7 10.0 mm to (128.3, 66.2), turned to 180 degrees
- moved JP3 5.15 mm to (132.6, 81.2)
- moved R5 3.84 mm to (118.2, 69.2)
- moved R8 2.90 mm to (118.2, 72.2)
- moved U1 1.95 mm to (139.3, 74.0)
- moved R9 1.47 mm to (118.2, 75.2)
- moved JP4 0.97 mm to (132.7, 83.8)
- moved C11 0.50 mm to (119.8, 78.2)
- moved Q13 0.25 mm to (163.8, 120.5)
- moved Q14 0.25 mm to (165.6, 117.1)
- moved Q15 0.25 mm to (167.8, 121.0)
- moved C2 0.21 mm to (137.0, 69.8)
Connections:
- U3 pad 2: 3V3 -> Net-(JP9-A)
Routing:
- net Net-(JP9-A): track 0.00 -> 37.3 mm
- net Vmid: track 74.8 -> 66.1 mm
- net Net-(R7-Pad1): track 15.5 -> 23.2 mm
- net 3V3: track 76.0 -> 81.8 mm
- net GND: track 61.6 -> 63.0 mm, vias 142 -> 172
- net Net-(JP3-A): track 10.9 -> 9.74 mm
- net Net-(U2-Vfb): track 22.5 -> 23.6 mm
- net 12V: track 199.8 -> 198.9 mm

Commit message: Board update
Routing:
- net GND: vias 172 -> 184
Changed lines of the file:
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@@
 		(tags "Through hole socket strip THT 2x05 2.54mm double row")
 		(property "Reference" "J1"
-			(at -3.58 12.25 0)
+			(at -0.58 12.5 0)
 			(layer "F.SilkS")
 			(effects
@@
 	)
 	(via
+		(at 119.899787 115.747597)
+		(size 0.6)
+		(drill 0.3)
+		(layers "F.Cu" "B.Cu")
+		(free yes)
+		(net 1)
+	)
+	(via
 		(at 165.5 85)
 		(size 0.6)
@@
 	)
 	(via
+		(at 121.399787 114.997597)
+		(size 0.6)
+		(drill 0.3)
+		(layers "F.Cu" "B.Cu")
+		(free yes)
+		(net 1)
+	)
+	(via
 		(at 147.25 90.25)
 		(size 0.6)
@@
 	)
 	(via
+		(at 121.399787 116.497597)
+		(size 0.6)
+		(drill 0.3)
+		(layers "F.Cu" "B.Cu")
+		(free yes)
+		(net 1)
+	)
+	(via
 		(at 130.75 92)
 		(size 0.6)
@@
 	)
 	(via
+		(at 120.649787 116.497597)
+		(size 0.6)
+		(drill 0.3)
+		(layers "F.Cu" "B.Cu")
+		(free yes)
+		(net 1)
+	)
+	(via
 		(at 137 84.25)
 		(size 0.6)
@@
 	)
 	(via
+		(at 121.399787 114.247597)
+		(size 0.6)
+		(drill 0.3)
+		(layers "F.Cu" "B.Cu")
+		(free yes)
+		(net 1)
+	)
+	(via
 		(at 153.75 89.5)
 		(size 0.6)
@@
 	)
 	(via
+		(at 120.649787 115.747597)
+		(size 0.6)
+		(drill 0.3)
+		(layers "F.Cu" "B.Cu")
+		(free yes)
+		(net 1)
+	)
+	(via
 		(at 157.25 102.25)
 		(size 0.6)
@@
 	)
 	(via
+		(at 119.899787 116.497597)
+		(size 0.6)
+		(drill 0.3)
+		(layers "F.Cu" "B.Cu")
+		(free yes)
+		(net 1)
+	)
+	(via
 		(at 141.75 97)
 		(size 0.6)
@@
 	)
 	(via
+		(at 120.649787 114.247597)
+		(size 0.6)
+		(drill 0.3)
+		(layers "F.Cu" "B.Cu")
+		(free yes)
+		(net 1)
+	)
+	(via
 		(at 135.5 79.25)
 		(size 0.6)
@@
 	)
 	(via
+		(at 120.649787 114.997597)
+		(size 0.6)
+		(drill 0.3)
+		(layers "F.Cu" "B.Cu")
+		(free yes)
+		(net 1)
+	)
+	(via
 		(at 137 83.5)
 		(size 0.6)
@@
 	)
 	(via
+		(at 119.899787 114.247597)
+		(size 0.6)
+		(drill 0.3)
+		(layers "F.Cu" "B.Cu")
+		(free yes)
+		(net 1)
+	)
+	(via
 		(at 162.5 86.5)
 		(size 0.6)
@@
 	)
 	(via
+		(at 121.399787 115.747597)
+		(size 0.6)
+		(drill 0.3)
+		(layers "F.Cu" "B.Cu")
+		(free yes)
+		(net 1)
+	)
+	(via
 		(at 143.25 100.75)
 		(size 0.6)
@@
 		(size 0.6)
 		(drill 0.3)
+		(layers "F.Cu" "B.Cu")
+		(free yes)
+		(net 1)
+	)
+	(via
+		(at 119.899787 114.997597)
+		(size 0.6)
+		(drill 0.3)
